File: bridge_rectifier.sch (KiCad schematic (older format))
At the start: 18 parts, among them P1 AC_INPUT, P2 OUTPUT, P3 MOUNTING_HOLES, P4 MOUNTING_HOLES, P5 MOUNTING_HOLES, P6 MOUNTING_HOLES

Commit message: trying to route the board within sqrt(2500)
Parts:
- removed P1: AC_INPUT, symbol CONN_01X03
- removed P2: OUTPUT, symbol CONN_01X03
- added P1: AC_INPUT, w_conn_screw:mstbva_2,5%2f2-g-5,08, symbol CONN_01X02
- added P2: OUTPUT, w_conn_screw:mstbva_2,5%2f2-g-5,08, symbol CONN_01X02
- C1: footprint (none) -> Capacitors_ThroughHole:C_Disc_D7.5_P5
- D1: footprint (none) -> w_pth_diodes:diode_do35
- D2: footprint (none) -> LEDs:LED-3MM
- D3, D4, D5, D6: footprint Diodes_ThroughHole:Diode_TO-220_Vertical -> jjrh_custom:MUR860
- P3, P4, P5, P6: footprint (none) -> mechanical:3.5mm_m3
- R1: footprint (none) -> w_pth_resistors:R12x5.2_vert
Connections:
- net HOT: now also P1.1 (P1)
- net Netural: now also P1.2 (P2)
- net V+: now also P2.1 (P1)
- net V-: now also P2.2 (P2)
Changed lines of the file:
@@
 LIBS:contrib
 LIBS:valves
-LIBS:linear_psu_v1-cache
-LIBS:5V_PSU-cache
-LIBS:powersupply_5v_v1-cache
+LIBS:bridge_rectifier-cache
 EELAYER 25 0
 EELAYER END
@@
 F 0 "D4" H 7430 2525 50  0000 C CNN
 F 1 "MUR860G" H 7430 2325 50  0000 C CNN
-F 2 "Diodes_ThroughHole:Diode_TO-220_Vertical" H 7430 2425 60  0001 C CNN
+F 2 "jjrh_custom:MUR860" H 7430 2425 60  0001 C CNN
 F 3 "" H 7430 2425 60  0000 C CNN
 F 4 "~" H 7430 2425 60  0000 C CNN "MANUFACTURER_PART"
@@
 F 0 "D3" H 7155 2875 50  0000 C CNN
 F 1 "MUR860G" H 7155 2675 50  0000 C CNN
-F 2 "Diodes_ThroughHole:Diode_TO-220_Vertical" H 7155 2775 60  0001 C CNN
+F 2 "jjrh_custom:MUR860" H 7155 2775 60  0001 C CNN
 F 3 "" H 7155 2775 60  0000 C CNN
 F 4 "~" H 7155 2775 60  0000 C CNN "MANUFACTURER_PART"
@@
 F 0 "D6" H 7705 2875 50  0000 C CNN
 F 1 "MUR860G" H 7705 2675 50  0000 C CNN
-F 2 "Diodes_ThroughHole:Diode_TO-220_Vertical" H 7705 2775 60  0001 C CNN
+F 2 "jjrh_custom:MUR860" H 7705 2775 60  0001 C CNN
 F 3 "" H 7705 2775 60  0000 C CNN
 F 4 "~" H 7705 2775 60  0000 C CNN "MANUFACTURER_PART"
@@
 F 0 "D5" H 7430 3175 50  0000 C CNN
 F 1 "MUR860G" H 7430 2975 50  0000 C CNN
-F 2 "Diodes_ThroughHole:Diode_TO-220_Vertical" H 7430 3075 60  0001 C CNN
+F 2 "jjrh_custom:MUR860" H 7430 3075 60  0001 C CNN
 F 3 "" H 7430 3075 60  0000 C CNN
 F 4 "~" H 7430 3075 60  0000 C CNN "MANUFACTURER_PART"
@@
 Text Label 8455 2425 0    60   ~ 0
 V+
-Text Label 6560 1045 0    60   ~ 0
-EARTH
 $Comp
 L C_Small C3
@@
 	1    0    0    -1
 $EndComp
+Text Notes 3640 615  0    60   ~ 0
+LIVE POWER INDICATION
+Text Label 5925 2425 0    60   ~ 0
+HOT
+Text Label 5905 3225 0    60   ~ 0
+Netural
+Text Label 6505 980  0    60   ~ 0
+HOT
+Text Label 6500 1085 0    60   ~ 0
+Netural
+$Comp
+L LED D2
+U 1 1 569177D6
+P 5045 1130
+F 0 "D2" H 5045 1230 50  0000 C CNN
+F 1 "LED" H 5045 1030 50  0000 C CNN
+F 2 "LEDs:LED-3MM" H 5045 1130 60  0001 C CNN
+F 3 "" H 5045 1130 60  0000 C CNN
+	1    5045 1130
+	0    -1   -1   0
+$EndComp
+$Comp
+L D D1
+U 1 1 56917920
+P 4515 1165
+F 0 "D1" H 4515 1265 50  0000 C CNN
+F 1 "D" H 4515 1065 50  0000 C CNN
+F 2 "w_pth_diodes:diode_do35" H 4515 1165 60  0001 C CNN
+F 3 "" H 4515 1165 60  0000 C CNN
+	1    4515 1165
+	0    1    1    0
+$EndComp
+$Comp
+L C C1
+U 1 1 56917AEF
+P 4015 835
+F 0 "C1" H 4040 935 50  0000 L CNN
+F 1 "C" H 4040 735 50  0000 L CNN
+F 2 "Capacitors_ThroughHole:C_Disc_D7.5_P5" H 4053 685 30  0001 C CNN
+F 3 "" H 4015 835 60  0000 C CNN
+	1    4015 835
+	0    1    1    0
+$EndComp
+Text Label 3300 835  0    60   ~ 0
+HOT
+Text Label 3295 1450 0    60   ~ 0
+Netural
+$Comp
+L R R1
+U 1 1 56917FA6
+P 4040 1450
+F 0 "R1" V 4120 1450 50  0000 C CNN
+F 1 "R" V 4040 1450 50  0000 C CNN
+F 2 "w_pth_resistors:R12x5.2_vert" V 3970 1450 30  0001 C CNN
+F 3 "" H 4040 1450 30  0000 C CNN
+	1    4040 1450
+	0    1    1    0
+$EndComp
+$Comp
+L CONN_01X01 P5
+U 1 1 56919752
+P 10630 935
+F 0 "P5" H 10630 1035 50  0000 C CNN
+F 1 "MOUNTING_HOLES" V 10730 935 50  0000 C CNN
+F 2 "mechanical:3.5mm_m3" H 10630 935 60  0001 C CNN
+F 3 "" H 10630 935 60  0000 C CNN
+	1    10630 935
+	0    1    1    0
+$EndComp
+$Comp
+L CONN_01X01 P6
+U 1 1 56919883
+P 10645 1530
+F 0 "P6" H 10645 1630 50  0000 C CNN
+F 1 "MOUNTING_HOLES" V 10745 1530 50  0000 C CNN
+F 2 "mechanical:3.5mm_m3" H 10645 1530 60  0001 C CNN
+F 3 "" H 10645 1530 60  0000 C CNN
+	1    10645 1530
+	0    1    1    0
+$EndComp
+$Comp
+L CONN_01X01 P4
+U 1 1 5691999F
+P 9930 950
+F 0 "P4" H 9930 1050 50  0000 C CNN
+F 1 "MOUNTING_HOLES" V 10030 950 50  0000 C CNN
+F 2 "mechanical:3.5mm_m3" H 9930 950 60  0001 C CNN
+F 3 "" H 9930 950 60  0000 C CNN
+	1    9930 950
+	0    1    1    0
+$EndComp
+$Comp
+L CONN_01X01 P3
+U 1 1 56919AC4
+P 9885 1520
+F 0 "P3" H 9885 1620 50  0000 C CNN
+F 1 "MOUNTING_HOLES" V 9985 1520 50  0000 C CNN
+F 2 "mechanical:3.5mm_m3" H 9885 1520 60  0001 C CNN
+F 3 "" H 9885 1520 60  0000 C CNN
+	1    9885 1520
+	0    1    1    0
+$EndComp
+NoConn ~ 10645 1330
+NoConn ~ 9885 1320
+NoConn ~ 9930 750
+NoConn ~ 10630 735
+Text Notes 6580 695  0    60   ~ 12
+120V INPUT
+Text Notes 8155 725  0    60   ~ 12
+RECTIFED OUTPUT
+$Comp
+L CONN_01X02 P1
+U 1 1 5691C944
+P 6995 1055
+F 0 "P1" H 6995 1205 50  0000 C CNN
+F 1 "AC_INPUT" V 7095 1055 50  0000 C CNN
+F 2 "w_conn_screw:mstbva_2,5%2f2-g-5,08" H 6995 1055 60  0001 C CNN
+F 3 "" H 6995 1055 60  0000 C CNN
+	1    6995 1055
+	1    0    0    -1
+$EndComp
 Wire Wire Line
 	5925 2425 7280 2425
@@
 Wire Notes Line
 	8280 2550 8280 2475
-Text Notes 3640 615  0    60   ~ 0
-LIVE POWER INDICATION
-$Comp
-L CONN_01X03 P1
-U 1 1 56914445
-P 6995 1050
-F 0 "P1" H 6995 1250 50  0000 C CNN
-F 1 "AC_INPUT" V 7095 1050 50  0000 C CNN
-F 2 "" H 6995 1050 60  0000 C CNN
-F 3 "" H 6995 1050 60  0000 C CNN
-	1    6995 1050
-	1    0    0    -1
-$EndComp
-Wire Wire Line
-	6795 1050 6560 1050
-Wire Wire Line
-	6560 1050 6560 1045
-Text Label 5925 2425 0    60   ~ 0
-HOT
-Text Label 5905 3225 0    60   ~ 0
-Netural
-Text Label 6560 940  0    60   ~ 0
-HOT
-Text Label 6500 1135 0    60   ~ 0
-Netural
-Wire Wire Line
-	6795 1150 6500 1150
-Wire Wire Line
-	6500 1150 6500 1135
-Wire Wire Line
-	6795 950  6560 950
-Wire Wire Line
-	6560 950  6560 940
-$Comp
-L LED D2
-U 1 1 569177D6
-P 5045 1130
-F 0 "D2" H 5045 1230 50  0000 C CNN
-F 1 "LED" H 5045 1030 50  0000 C CNN
-F 2 "" H 5045 1130 60  0000 C CNN
-F 3 "" H 5045 1130 60  0000 C CNN
-	1    5045 1130
-	0    -1   -1   0
-$EndComp
-$Comp
-L D D1
-U 1 1 56917920
-P 4515 1165
-F 0 "D1" H 4515 1265 50  0000 C CNN
-F 1 "D" H 4515 1065 50  0000 C CNN
-F 2 "" H 4515 1165 60  0000 C CNN
-F 3 "" H 4515 1165 60  0000 C CNN
-	1    4515 1165
-	0    1    1    0
-$EndComp
-$Comp
-L C C1
-U 1 1 56917AEF
-P 4015 835
-F 0 "C1" H 4040 935 50  0000 L CNN
-F 1 "C" H 4040 735 50  0000 L CNN
-F 2 "" H 4053 685 30  0000 C CNN
-F 3 "" H 4015 835 60  0000 C CNN
-	1    4015 835
-	0    1    1    0
-$EndComp
-Text Label 3300 835  0    60   ~ 0
-HOT
-Text Label 3295 1450 0    60   ~ 0
-Netural
 Wire Wire Line
 	3865 835  3300 835
@@
 Wire Wire Line
 	5045 835  5045 930
-$Comp
-L R R1
-U 1 1 56917FA6
-P 4040 1450
-F 0 "R1" V 4120 1450 50  0000 C CNN
-F 1 "R" V 4040 1450 50  0000 C CNN
-F 2 "" V 3970 1450 30  0000 C CNN
-F 3 "" H 4040 1450 30  0000 C CNN
-	1    4040 1450
-	0    1    1    0
-$EndComp
 Wire Wire Line
 	4190 1450 5045 1450
@@
 Wire Wire Line
 	3295 1450 3890 1450
-$Comp
-L CONN_01X03 P2
-U 1 1 56918D5B
-P 8760 1090
-F 0 "P2" H 8760 1290 50  0000 C CNN
-F 1 "OUTPUT" V 8860 1090 50  0000 C CNN
-F 2 "" H 8760 1090 60  0000 C CNN
-F 3 "" H 8760 1090 60  0000 C CNN
-	1    8760 1090
+Wire Notes Line
+	4730 575  5340 575
+Wire Notes Line
+	5340 575  5340 1730
+Wire Notes Line
+	5340 1730 3045 1730
+Wire Notes Line
+	3045 1730 3045 575
+Wire Notes Line
+	3045 575  3605 575
+Wire Notes Line
+	9285 525  9285 1875
+Wire Notes Line
+	9285 1875 11155 1875
+Wire Notes Line
+	7275 700  7275 1450
+Wire Notes Line
+	7275 1450 6345 1450
+Wire Notes Line
+	6345 1450 6345 695
+Wire Notes Line
+	6345 695  6475 695
+Wire Notes Line
+	8990 675  8990 1320
+Wire Notes Line
+	8990 1320 8040 1320
+Wire Notes Line
+	8040 1320 8040 680
+Wire Notes Line
+	8040 680  8135 680
+Wire Notes Line
+	8990 675  8960 675
+Wire Wire Line
+	6795 1005 6505 1005
+Wire Wire Line
+	6505 1005 6505 980
+Wire Wire Line
+	6795 1105 6500 1105
+Wire Wire Line
+	6500 1105 6500 1085
+$Comp
+L CONN_01X02 P2
+U 1 1 5691D34D
+P 8640 1030
+F 0 "P2" H 8640 1180 50  0000 C CNN
+F 1 "OUTPUT" V 8740 1030 50  0000 C CNN
+F 2 "w_conn_screw:mstbva_2,5%2f2-g-5,08" H 8640 1030 60  0001 C CNN
+F 3 "" H 8640 1030 60  0000 C CNN
+	1    8640 1030
 	1    0    0    -1
 $EndComp
-Text Label 8215 955  0    60   ~ 0
+Text Label 8275 980  0    60   ~ 0
 V+
-Text Label 8220 1190 0    60   ~ 0
+Wire Wire Line
+	8440 980  8275 980
+Text Label 8290 1075 0    60   ~ 0
 V-
 Wire Wire Line
-	8220 1190 8560 1190
-Wire Wire Line
-	8215 955  8560 955
-Wire Wire Line
-	8560 955  8560 990
-Text Label 8215 1090 0    60   ~ 0
-EARTH
-Wire Wire Line
-	8215 1090 8560 1090
-Wire Notes Line
-	4730 575  5340 575
-Wire Notes Line
-	5340 575  5340 1730
-Wire Notes Line
-	5340 1730 3045 1730
-Wire Notes Line
-	3045 1730 3045 575
-Wire Notes Line
-	3045 575  3605 575
-$Comp
-L CONN_01X01 P5
-U 1 1 56919752
-P 10630 935
-F 0 "P5" H 10630 1035 50  0000 C CNN
-F 1 "MOUNTING_HOLES" V 10730 935 50  0000 C CNN
-F 2 "" H 10630 935 60  0000 C CNN
-F 3 "" H 10630 935 60  0000 C CNN
-	1    10630 935
-	0    1    1    0
-$EndComp
-$Comp
-L CONN_01X01 P6
-U 1 1 56919883
-P 10645 1530
-F 0 "P6" H 10645 1630 50  0000 C CNN
-F 1 "MOUNTING_HOLES" V 10745 1530 50  0000 C CNN
-F 2 "" H 10645 1530 60  0000 C CNN
-F 3 "" H 10645 1530 60  0000 C CNN
-	1    10645 1530
-	0    1    1    0
-$EndComp
-$Comp
-L CONN_01X01 P4
-U 1 1 5691999F
-P 9930 950
-F 0 "P4" H 9930 1050 50  0000 C CNN
-F 1 "MOUNTING_HOLES" V 10030 950 50  0000 C CNN
-F 2 "" H 9930 950 60  0000 C CNN
-F 3 "" H 9930 950 60  0000 C CNN
-	1    9930 950
-	0    1    1    0
-$EndComp
-$Comp
-L CONN_01X01 P3
-U 1 1 56919AC4
-P 9885 1520
-F 0 "P3" H 9885 1620 50  0000 C CNN
-F 1 "MOUNTING_HOLES" V 9985 1520 50  0000 C CNN
-F 2 "" H 9885 1520 60  0000 C CNN
-F 3 "" H 9885 1520 60  0000 C CNN
-	1    9885 1520
-	0    1    1    0
-$EndComp
-NoConn ~ 10645 1330
-NoConn ~ 9885 1320
-NoConn ~ 9930 750
-NoConn ~ 10630 735
-Wire Notes Line
-	9285 525  9285 1875
-Wire Notes Line
-	9285 1875 11155 1875
-Wire Notes Line
-	7275 700  7275 1450
-Wire Notes Line
-	7275 1450 6345 1450
-Wire Notes Line
-	6345 1450 6345 695
-Wire Notes Line
-	6345 695  6475 695
-Text Notes 6580 695  0    60   ~ 12
-120V INPUT
-Text Notes 8155 725  0    60   ~ 12
-RECTIFED OUTPUT
-Wire Notes Line
-	8990 675  8990 1320
-Wire Notes Line
-	8990 1320 8040 1320
-Wire Notes Line
-	8040 1320 8040 680
-Wire Notes Line
-	8040 680  8135 680
-Wire Notes Line
-	8990 675  8960 675
+	8440 1080 8290 1080
+Wire Wire Line
+	8290 1080 8290 1075
 $EndSCHEMATC
