File: bridge_rectifier.kicad_pcb (KiCad board)
At the start: 2 copper layers, 122.7 x 95.6 mm, 18 parts, among them P1 AC_INPUT, P2 OUTPUT, P3 MOUNTING_HOLES, P4 MOUNTING_HOLES, P5 MOUNTING_HOLES, P6 MOUNTING_HOLES

Commit message: routed final
Parts:
- moved D2 194.9 mm to (265.5, 115.6)
- moved R1 183.9 mm to (248.3, 117.3), turned to 90 degrees
- moved D1 183.6 mm to (260.3, 115.3), turned to 90 degrees
- moved P3 179.6 mm to (270.1, 117.8)
- moved P6 175.0 mm to (270.1, 76.6)
- moved C1 172.0 mm to (254.9, 117.7), turned to 90 degrees
- moved P1 149.4 mm to (237.2, 115.3), turned to 0 degrees
- moved D3 115.3 mm to (255.2, 107.5), turned to 0 degrees
- moved D4 114.6 mm to (219.0, 107.5), turned to 0 degrees
- moved C3 112.2 mm to (221.5, 99.9), turned to 180 degrees
- moved C2 103.9 mm to (252.7, 99.9), turned to 0 degrees
- moved D5 103.6 mm to (255.2, 93.2), turned to 0 degrees
- moved D6 102.8 mm to (219.0, 93.3), turned to 0 degrees
- moved C4 95.0 mm to (252.7, 85.6), turned to 0 degrees
- moved C5 94.2 mm to (216.5, 85.7), turned to 0 degrees
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Routing:
- net (no net): track 529.8 -> 0.00 mm, vias 2 -> 0
- net /HOT: track 7.04 -> 62.5 mm
- net /V+: track 0.00 -> 44.6 mm
- net /V-: track 0.00 -> 44.3 mm
- net Net-(D1-Pad2): track 11.7 -> 23.5 mm
- net /Netural: track 89.1 -> 77.4 mm, vias 0 -> 1
- net Net-(C1-Pad1): track 17.6 -> 10.7 mm
Other:
- board size 122.7 x 95.6 mm -> 71.8 x 47.1 mm

Commit message: added highvoltage symbol
Parts:
- added REF**: Symbol_HighVoltage_Type2_CopperTop_VerySmall, Symbols:Symbol_HighVoltage_Type2_CopperTop_VerySmall, F.Cu at (225.5, 117.0)
Changed lines of the file:
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@@
   (general
     (links 22)
-    (no_connects 22)
-    (area -53.871601 43.754699 204.342 161.526201)
+    (no_connects 0)
+    (area 201.118795 73.432869 273.150001 120.77551)
     (thickness 1.6)
     (drawings 4)
     (tracks 71)
     (zones 0)
-    (modules 18)
+    (modules 19)
     (nets 7)
   )
@@
     )
   )
+  (module Symbols:Symbol_HighVoltage_Type2_CopperTop_VerySmall (layer F.Cu)
+    (at 225.5012 117.0178)
+    (descr "Symbol, High Voltage, Type 2, Copper Top, Very Small,")
+    (tags "Symbol, High Voltage, Type 2, Copper Top, Very Small,")
+    (fp_text reference REF** (at -0.1524 0.7112) (layer F.SilkS) hide
+      (effects (font (size 1 1) (thickness 0.15)))
+    )
+    (fp_text value Symbol_HighVoltage_Type2_CopperTop_VerySmall (at -0.381 4.572) (layer F.Fab) hide
+      (effects (font (size 1 1) (thickness 0.15)))
+    )
+    (fp_line (start -0.49784 2.19964) (end 0.70104 -0.89916) (layer F.Cu) (width 0.381))
+    (fp_line (start 0.70104 -0.89916) (end 0.1016 -0.50038) (layer F.Cu) (width 0.381))
+    (fp_line (start -0.89916 0.20066) (end 0.40132 -2.60096) (layer F.Cu) (width 0.381))
+    (fp_line (start -0.49784 2.19964) (end 0.1016 1.50114) (layer F.Cu) (width 0.381))
+    (fp_line (start -0.09906 -2.79908) (end -0.89916 0.20066) (layer F.Cu) (width 0.381))
+    (fp_line (start -0.89916 0.20066) (end 0.29972 -0.59944) (layer F.Cu) (width 0.381))
+    (fp_line (start 0.29972 -0.59944) (end -0.49784 2.19964) (layer F.Cu) (width 0.381))
+    (fp_line (start -0.49784 2.19964) (end -0.59944 1.30048) (layer F.Cu) (width 0.381))
+    (fp_line (start 0 -4.191) (end 4.699 2.794) (layer F.Cu) (width 0.381))
+    (fp_line (start 4.699 2.794) (end -4.699 2.794) (layer F.Cu) (width 0.381))
+    (fp_line (start -4.699 2.794) (end 0 -4.191) (layer F.Cu) (width 0.381))
+  )
   (gr_line (start 201.2188 120.675509) (end 201.2188 73.53287) (layer Edge.Cuts) (width 0.2))
